File: OBC/OBC.kicad_sch (KiCad schematic)
At the start: 11 parts, among them U1 LSM9DS1TR, U2 HTS221TR

Commit message: v0.3-pcb ok
Parts:
- added H1, H2, H3, H4, H5, H6: 1, MountingHole:MountingHole_2.7mm_M2.5_Pad_Via, symbol Mechanical:MountingHole_Pad
- R1: footprint OptoDevice:R_LDR_4.9x4.2mm_P2.54mm_Vertical -> Resistor_SMD:R_0201_0603Metric
Connections:
- net +3V3: now also C7.1; no longer C7.2
- net GND: now also C7.2, U2.5 (GND), H1.1, H2.1, H3.1, H4.1, H5.1, H6.1
